Commit message: lab1_solution

File: src/urdf_demo/urdf/robot.urdf (robot description, URDF)
Before this commit: robot robot, 2 links, 1 joints
Links:
- added link slider_link, mass 0.5; collision box size=0.5 0.25 0.15; visual box size=0.5 0.25 0.15
Joints:
- added joint slider_joint: type prismatic, parent base_link, child slider_link, origin xyz=-1.25 0 0.1 rpy=0 0 0, axis 1 0 0, limit lower=0 upper=2 effort=100 velocity=100
