Commit message: add camera sensor

File: src/urdf_demo/urdf/gazebo.xacro (robot description, xacro)
@@ -24,3 +24,35 @@
         </plugin>
     </gazebo>
+    <joint name="camera_optical_joint" type="fixed">
+        <origin xyz="0 0 0" rpy="-1.571 0 -1.571" />
+        <parent link="camera_link" />
+        <child link="camera_link_optical" />
+    </joint>
+    <link name="camera_link_optical"></link>
+    <gazebo reference="camera_link">
+        <sensor type="camera" name="my_camera">
+            <update_rate>20</update_rate>
+            <visualize>true</visualize>
+            <camera name="cam">
+                <horizontal_fov>1.3962634</horizontal_fov>
+                <image>
+                    <width>640</width>
+                    <height>480</height>
+                    <format>R8G8B8</format>
+                </image>
+                <clip>
+                    <near>0.02</near>
+                    <far>300</far>
+                </clip>
+                <noise>
+                    <type>gaussian</type>
+                    <mean>0.0</mean>
+                    <stddev>0.007</stddev>
+                </noise>
+            </camera>
+            <plugin name="camera_controller" filename="libgazebo_ros_camera.so">
+                <frame_name>camera_link_optical</frame_name>
+            </plugin>
+        </sensor>
+    </gazebo>
 </robot>

Commit message: add ir sensor

File: src/urdf_demo/urdf/gazebo.xacro (robot description, xacro)
@@ -56,3 +56,65 @@
         </sensor>
     </gazebo>
+    <link name="ir_link">
+        <origin xyz="${arm_length} 0 ${arm_radius - 0.075}" rpy="0 0 0"/>
+        <collision>
+          <origin xyz="0 0 0" rpy="0 0 0"/>
+          <geometry>
+            <box size="0.01 0.01 0.01"/>
+          </geometry>
+        </collision>    <visual>
+          <origin xyz="0 0 0" rpy="0 0 0"/>
+          <geometry>
+            <box size="0.01 0.01 0.01"/>
+          </geometry>
+          <material name="black">
+            <color rgba="0 0 0 1"/>
+        </material>
+        </visual>
+        <xacro:inertial_box mass="1e-5" x="0.01" y="0.01" z="0.01">
+            <origin xyz="0.0 0 0" rpy="0 0 0"/>
+        </xacro:inertial_box>
+    </link>
+    <joint name="ir_joint" type="fixed">
+        <origin xyz="0 0 0" rpy="0 1.571 0"/>
+        <parent link="arm_link"/>
+        <child link="ir_link"/>
+    </joint>
+    <gazebo reference="ir_link">
+        <sensor type="ray" name="TeraRanger">
+           <pose>0 0 0 0 0 0</pose>
+           <visualize>true</visualize>
+           <update_rate>50</update_rate>
+           <ray>
+              <scan>
+                 <horizontal>
+                    <samples>10</samples>
+                    <resolution>1</resolution>
+                    <min_angle>-0.14835</min_angle>
+                    <max_angle>0.14835</max_angle>
+                 </horizontal>
+                 <vertical>
+                    <samples>10</samples>
+                    <resolution>1</resolution>
+                    <min_angle>-0.14835</min_angle>
+                    <max_angle>0.14835</max_angle>
+                 </vertical>
+              </scan>
+              <range>
+                 <min>0.01</min>
+                 <max>2</max>
+                 <resolution>0.02</resolution>
+              </range>
+           </ray>
+           <plugin filename="libgazebo_ros_ray_sensor.so" name="gazebo_ros_range">
+              <gaussianNoise>0.005</gaussianNoise>
+              <alwaysOn>true</alwaysOn>
+              <updateRate>50</updateRate>
+              <topicName>sensor/ir_front</topicName>
+              <frameName>ir_link</frameName>
+              <radiation>INFRARED</radiation>
+              <fov>0.2967</fov>
+           </plugin>
+        </sensor>
+        </gazebo>
 </robot>

File: src/urdf_demo/urdf/robot.xacro (robot description, xacro)
@@ -1,8 +1,8 @@
 <?xml version="1.0"?>
 <robot xmlns:xacro="http://www.ros.org/wiki/xacro" name="robot">
+    <xacro:property name="arm_length" value="1" />
+    <xacro:property name="arm_radius" value="0.1" />
     <xacro:include filename="utils.xacro" />
     <xacro:include filename="gazebo.xacro" />
-    <xacro:property name="arm_length" value="1" />
-    <xacro:property name="arm_radius" value="0.1" />
     <link name="world"></link>
     <joint name="base_joint" type="fixed">

Commit message: range ultrasonic

File: src/urdf_demo/urdf/gazebo.xacro (robot description, xacro)
@@ -11,6 +11,5 @@
     </gazebo>
     <gazebo>
-        <plugin name="gazebo_ros_joint_state_publisher"
-            filename="libgazebo_ros_joint_state_publisher.so">
+        <plugin name="gazebo_ros_joint_state_publisher" filename="libgazebo_ros_joint_state_publisher.so">
             <update_rate>20</update_rate>
             <joint_name>slider_joint</joint_name>
@@ -19,6 +18,5 @@
     </gazebo>
     <gazebo>
-        <plugin name="gazebo_ros_joint_pose_trajectory"
-            filename="libgazebo_ros_joint_pose_trajectory.so">
+        <plugin name="gazebo_ros_joint_pose_trajectory" filename="libgazebo_ros_joint_pose_trajectory.so">
             <update_rate>20</update_rate>
         </plugin>
@@ -57,18 +55,19 @@
     </gazebo>
     <link name="ir_link">
-        <origin xyz="${arm_length} 0 ${arm_radius - 0.075}" rpy="0 0 0"/>
         <collision>
-          <origin xyz="0 0 0" rpy="0 0 0"/>
-          <geometry>
-            <box size="0.01 0.01 0.01"/>
-          </geometry>
-        </collision>    <visual>
-          <origin xyz="0 0 0" rpy="0 0 0"/>
-          <geometry>
-            <box size="0.01 0.01 0.01"/>
-          </geometry>
-          <material name="black">
-            <color rgba="0 0 0 1"/>
-        </material>
+            <origin xyz="0 0 0" rpy="0 0 0"/>
+            <geometry>
+                <box size="0.01 0.01 0.01"/>
+            </geometry>
+        </collision>
+        <visual>
+            <origin xyz="0 0 0" rpy="0 0 0"/>
+            <origin xyz="0 0 0" rpy="0 0 0"/>
+            <geometry>
+                <box size="0.01 0.01 0.01"/>
+            </geometry>
+            <material name="black">
+                <color rgba="0 0 0 1"/>
+            </material>
         </visual>
         <xacro:inertial_box mass="1e-5" x="0.01" y="0.01" z="0.01">
@@ -77,44 +76,43 @@
     </link>
     <joint name="ir_joint" type="fixed">
-        <origin xyz="0 0 0" rpy="0 1.571 0"/>
+        <origin xyz="${arm_length} 0 -${arm_radius}" rpy="0 1.575 0"/>
         <parent link="arm_link"/>
         <child link="ir_link"/>
     </joint>
     <gazebo reference="ir_link">
-        <sensor type="ray" name="TeraRanger">
-           <pose>0 0 0 0 0 0</pose>
-           <visualize>true</visualize>
-           <update_rate>50</update_rate>
-           <ray>
-              <scan>
-                 <horizontal>
-                    <samples>10</samples>
-                    <resolution>1</resolution>
-                    <min_angle>-0.14835</min_angle>
-                    <max_angle>0.14835</max_angle>
-                 </horizontal>
-                 <vertical>
-                    <samples>10</samples>
-                    <resolution>1</resolution>
-                    <min_angle>-0.14835</min_angle>
-                    <max_angle>0.14835</max_angle>
-                 </vertical>
-              </scan>
-              <range>
-                 <min>0.01</min>
-                 <max>2</max>
-                 <resolution>0.02</resolution>
-              </range>
-           </ray>
-           <plugin filename="libgazebo_ros_ray_sensor.so" name="gazebo_ros_range">
-              <gaussianNoise>0.005</gaussianNoise>
-              <alwaysOn>true</alwaysOn>
-              <updateRate>50</updateRate>
-              <topicName>sensor/ir_front</topicName>
-              <frameName>ir_link</frameName>
-              <radiation>INFRARED</radiation>
-              <fov>0.2967</fov>
-           </plugin>
-        </sensor>
-        </gazebo>
+        <sensor type="ray" name="ultrasonic_sensor">
+            <pose>0 0 0 0 0 0</pose>
+            <visualize>true</visualize>
+            <update_rate>5</update_rate>
+            <ray>
+                <scan>
+                    <horizontal>
+                        <samples>5</samples>
+                        <resolution>1.000000</resolution>
+                        <min_angle>-0.12</min_angle>
+                        <max_angle>0.12</max_angle>
+                    </horizontal>
+                    <vertical>
+                        <samples>5</samples>
+                        <resolution>1.000000</resolution>
+                        <min_angle>-0.01</min_angle>
+                        <max_angle>0.01</max_angle>
+                    </vertical>
+                </scan>
+                <range>
+                    <min>0.01</min>
+                    <max>2</max>
+                    <resolution>0.02</resolution>
+                </range>
+            </ray>
+            <plugin name="ultrasonic_plugin" filename="libgazebo_ros_ray_sensor.so">
+            <ros>
+                <remapping>~/out:=ultrasound/range</remapping>
+            </ros>
+            <output_type>sensor_msgs/Range</output_type>
+            <radiation_type>ultrasound</radiation_type>
+            <frame_name>ir_link</frame_name>
+        </plugin>
+    </sensor>
+</gazebo>
 </robot>
