Commit message: add imu state broadcaster

File: src/urdf_demo/urdf/imu.urdf.xacro (robot description, xacro)
@@ -21,5 +21,5 @@
                 <box size="0.02 0.02 0.02"/>
             </geometry>
-            <material name="iRobot/Red"/>
+            <material name="red"/>
         </visual>
         <inertial>

File: src/urdf_demo/urdf/ros_control_velocity.urdf.xacro (robot description, xacro)
@@ -8,5 +8,4 @@
         <joint name="slider_joint">
             <command_interface name="velocity"/>
-            <state_interface name="position"/>
             <state_interface name="velocity"/>
             <state_interface name="position"/>
@@ -18,4 +17,16 @@
             <state_interface name="effort"/>
         </joint>
+        <sensor name="imu_sensor">
+            <state_interface name="orientation.x"/>
+            <state_interface name="orientation.y"/>
+            <state_interface name="orientation.z"/>
+            <state_interface name="orientation.w"/>
+            <state_interface name="angular_velocity.x"/>
+            <state_interface name="angular_velocity.y"/>
+            <state_interface name="angular_velocity.z"/>
+            <state_interface name="linear_acceleration.x"/>
+            <state_interface name="linear_acceleration.y"/>
+            <state_interface name="linear_acceleration.z"/>
+          </sensor>
     </ros2_control>
     <gazebo>

File: src/urdf_demo/urdf/utils.xacro (robot description, xacro)
@@ -6,4 +6,7 @@
     <material name="white">
         <color rgba="1 1 1 1"/>
+    </material>
+    <material name="red">
+        <color rgba="1 0 0 1"/>
     </material>
     <material name="orange">
