Commit message: lab3  exercise 01

File: src/urdf_demo/urdf/robot.xacro (robot description, xacro)
@@ -2,7 +2,7 @@
 <robot xmlns:xacro="http://www.ros.org/wiki/xacro" name="robot">
     <xacro:include filename="utils.xacro" />
+    <xacro:include filename="gazebo.xacro" />
     <xacro:property name="arm_length" value="1" />
     <xacro:property name="arm_radius" value="0.1" />
-    <xacro:arg name="color" default="blue"/>
     <link name="world"></link>
     <joint name="base_joint" type="fixed">
@@ -36,4 +36,5 @@
         <child link="slider_link"/>
         <axis xyz="1 0 0"/>
+        <dynamics damping="10.0" friction="10.0"/>
         <limit lower="0" upper="2" velocity="100" effort="100"/>
     </joint>
@@ -44,5 +45,5 @@
                 <box size="0.5 0.25 0.15" />
             </geometry>
-            <material name="$(arg color)" />
+            <material name="blue" />
         </visual>
         <collision>
@@ -61,4 +62,5 @@
         <child link="arm_link"/>
         <axis xyz="0 -1 0"/>
+        <dynamics damping="10.0" friction="10.0"/>
         <limit lower="0" upper="${pi/2}" velocity="100" effort="100"/>
     </joint>

Commit message: imu sensor

File: src/urdf_demo/urdf/robot.xacro (robot description, xacro)
@@ -5,4 +5,5 @@
     <xacro:include filename="utils.xacro" />
     <xacro:include filename="gazebo.xacro" />
+    <xacro:include filename="imu.urdf.xacro" />
     <link name="world"></link>
     <joint name="base_joint" type="fixed">

File: src/urdf_demo/urdf/utils.xacro (robot description, xacro)
@@ -1,4 +1,7 @@
 <?xml version="1.0"?>
 <robot xmlns:xacro="http://www.ros.org/wiki/xacro">
+    <material name="black">
+        <color rgba="0 0 0 1"/>
+    </material>
     <material name="white">
         <color rgba="1 1 1 1"/>

Commit message: bk

File: src/urdf_demo/urdf/robot.xacro (robot description, xacro)
@@ -1,15 +1,19 @@
 <?xml version="1.0"?>
 <robot xmlns:xacro="http://www.ros.org/wiki/xacro" name="robot">
-    <xacro:arg name="use_effort" default="false"/>
+    <xacro:arg name="type" default="position"/>
+    <xacro:property name="controller_type" value="$(arg type)" />
     <xacro:property name="arm_length" value="1" />
     <xacro:property name="arm_radius" value="0.1" />
     <xacro:include filename="utils.xacro" />
     <xacro:include filename="gazebo.xacro" />
-    <xacro:if value="$(arg use_effort)">
+    <xacro:if value="${controller_type == 'effort'}">
         <xacro:include filename="ros_control_effort.urdf.xacro" />
     </xacro:if>
-    <xacro:unless value="$(arg use_effort)">
+    <xacro:if value="${controller_type == 'position'}">
         <xacro:include filename="ros_control.urdf.xacro" />
-    </xacro:unless>
+    </xacro:if>
+    <xacro:if value="${controller_type == 'velocity'}">
+        <xacro:include filename="ros_control_velocity.urdf.xacro" />
+    </xacro:if>
     <xacro:include filename="imu.urdf.xacro" />
     <link name="world"></link>

Commit message: fix readme

File: src/urdf_demo/urdf/robot.xacro (robot description, xacro)
@@ -81,33 +81,3 @@
         </xacro:inertial_cylinder>
     </link>
-    <joint name="camera_joint" type="fixed">
-        <origin xyz="${arm_length} 0 ${arm_radius + 0.075}" rpy="0 0 0"/>
-        <parent link="arm_link"/>
-        <child link="camera_link"/>
-    </joint>
-    <link name="camera_link">
-        <visual>
-            <origin xyz="-0.03 0 0" rpy="0 0 0"/>
-            <geometry>
-                <box size="0.06 0.15 0.15" />
-            </geometry>
-            <material name="white" />
-        </visual>
-        <visual>
-            <origin xyz="0.03 0 0" rpy="0 ${pi/2} 0"/>
-            <geometry>
-                <cylinder length="0.06" radius="0.04" />
-            </geometry>
-            <material name="blue" />
-        </visual>
-        <collision>
-            <origin xyz="0.0 0 0" rpy="0 0 0"/>
-            <geometry>
-                <box size="0.12 0.15 0.15" />
-            </geometry>
-        </collision>
-        <xacro:inertial_box mass="0.1" x="0.12" y="0.15" z="0.15">
-            <origin xyz="0.0 0 0" rpy="0 0 0"/>
-        </xacro:inertial_box>
-    </link>
 </robot>

File: src/urdf_demo/urdf/utils.xacro (robot description, xacro)
@@ -7,6 +7,6 @@
         <color rgba="1 0.3 0.1 1"/>
     </material>
-    <material name="blue">
-        <color rgba="0.2 0.2 1 1"/>
+    <material name="black">
+        <color rgba="0 0 0 1"/>
     </material>
     <xacro:macro name="inertial_sphere" params="mass radius *origin">
